File: Hardware/PCB_2D.brd (EAGLE design)
At the start: 170.2 x 111.2 mm, 103 parts, among them IC1 BD5229G-TR, IC4 XC6220A331MR-G, J1 FH34SRJ-24S-0.5SH_99_, J2 SAMACSYS_PARTS_USB4110-GF-A, J3 QWIIC_RIGHT_ANGLE, J4 112A-TAAR-R03_ATTEND, Q1 20V/4.2A/52mΩ/1.4W, Q2 20V/4.2A/52mΩ/1.4W, Q3 SI1308EDL-T1-GE3, U1 W25Q512JVEIQ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

Commit message: Fixed issues
Parts:
- CHG_LED, SJ1: value (none) -> (none)
Connections:
- new net N$6: C_DELAY.1, IC1.5
- net 3V3: no longer C_DELAY.1, IC1.5, R_BOOT.1
- net IO/BOOT: now also R_BOOT.1
Routing:
- net GND: track 682.1 -> 632.6 mm, vias 13 -> 14
- net MISO: track 129.5 -> 103.2 mm, vias 4 -> 6
- net EPD_DC: track 142.3 -> 166.6 mm, vias 4 -> 3
- net SDA: track 215.4 -> 194.9 mm, vias 7 -> 6
- net EPD_RST: track 132.5 -> 150.5 mm, vias 4 -> 3
- net SCL: track 209.7 -> 191.8 mm, vias 6 -> 9
- net USB_D+: track 146.4 -> 155.6 mm, vias 2 -> 4
- net N$22: track 7.59 -> 16.6 mm, vias 0 -> 2
- net N$13: track 17.3 -> 25.9 mm, vias 0 -> 2
- net EPD_3V3_C: track 136.0 -> 127.5 mm, vias 3 -> 2
- net FLASH_CS: track 59.1 -> 51.3 mm, vias 0 -> 4
- net SCK: track 190.7 -> 197.1 mm, vias 12 -> 8
- net USB_D-: track 142.5 -> 148.5 mm
- net 32KHZ: track 86.9 -> 92.5 mm, vias 2 -> 4
- net IO/BOOT: track 61.5 -> 57.1 mm, vias 0 -> 5
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